File: esp32-circuit/untitled.kicad_sch (KiCad schematic)
At the start: 3 parts, among them SW1 SW_Push, U1 ESP32-S3-WROOM-1

Commit message: d00in
Parts:
- added SW3, SW4: SW_Push, symbol Switch:SW_Push
Connections:
- net GND: now also SW3.1, SW4.1
- net at U1.27 (IO0): now also SW4.2
- net at U1.3 (EN): now also SW3.2
